File: orca_keyboard/orca_keyboard.sch (KiCad schematic (older format))
At the start: 2 parts, among them U1 ProMicro

Commit message: .
Parts:
- removed K?1: KEYSW, symbol keyboard_parts:KEYSW
- removed U1: ProMicro, symbol promicro:ProMicro
- added B1: SPARKFUN_PRO_MICRO, Boards:SPARKFUN_PRO_MICRO, symbol SparkFun-Boards:SPARKFUN_PRO_MICRO
- added D00, D01, D02, D03, D04, D05, D06, D07, D10, D11, D12, D13, D14, D15, D16, D17, D22, D23, D24, D25: D, keyboard_parts:D_SOD123_axial, symbol keyboard_parts:D
- added K00, K01, K02, K03, K04, K05, K06, K07, K10, K11, K12, K13, K14, K15, K16, K17, K22, K23, K24, K25: KEYSW, keebs:Mx_Alps_100, symbol keyboard_parts:KEYSW
Connections:
- new net: D05.2, K05.2
- new net: D06.2, K06.2
- new net: D07.2, K07.2
- new net: D04.2, K04.2
- new net: D03.2, K03.2
- new net: D02.2, K02.2
- new net: D01.2, K01.2
- new net: D00.2, K00.2
- new net: D10.2, K10.2
- new net: D11.2, K11.2
- new net: D12.2, K12.2
- new net: D13.2, K13.2
- new net: D14.2, K14.2
- new net: D15.2, K15.2
- new net: D16.2, K16.2
- new net: D17.2, K17.2
- new net: D22.2, K22.2
- new net: D23.2, K23.2
- new net: D24.2, K24.2
- new net: D25.2, K25.2
- new net col0: B1.20 (A3), K00.1, K10.1
- new net col1: B1.19 (A2), K01.1, K11.1
- new net col2: B1.18 (A1), K02.1, K12.1, K22.1
- new net col3: B1.17 (A0), K03.1, K13.1, K23.1
- new net col4: B1.16 (13(SCK)), K04.1, K14.1, K24.1
- new net col5: B1.15 (12(MISO)), K05.1, K15.1, K25.1
- new net col6: B1.14 (11(MOSI)), K06.1, K16.1
- new net col7: B1.13 (*10), K07.1, K17.1
- new net row0: B1.10 (7), D00.1, D01.1, D02.1, D03.1, D04.1, D05.1, D06.1, D07.1
- new net row1: B1.11 (8), D10.1, D11.1, D12.1, D13.1, D14.1, D15.1, D16.1, D17.1
- new net row2: B1.12 (*9), D22.1, D23.1, D24.1, D25.1
