File: orca_keyboard/orca_keyboard.kicad_pcb (KiCad board)
At the start: 2 copper layers, 2 parts, among them U1 ProMicro

Commit message: .
Parts:
- removed K?1: KEYSW, keebs:Mx_Alps_100
- removed U1: ProMicro, promicro:ProMicro
- added B1: SPARKFUN_PRO_MICRO, Boards:SPARKFUN_PRO_MICRO, F.Cu at (261.2, -179.8)
- added D00: D, keyboard_parts:D_SOD123_axial, F.Cu at (336.7, -122.1)
- added D01: D, keyboard_parts:D_SOD123_axial, F.Cu at (357.5, -142.1)
- added D02: D, keyboard_parts:D_SOD123_axial, F.Cu at (336.7, -125.7)
- added D03: D, keyboard_parts:D_SOD123_axial, F.Cu at (356.6, -145.7)
- added D04: D, keyboard_parts:D_SOD123_axial, F.Cu at (376.6, -165.6)
- added D05: D, keyboard_parts:D_SOD123_axial, F.Cu at (347.1, -132.9)
- added D06: D, keyboard_parts:D_SOD123_axial, F.Cu at (387.0, -176.4)
- added D07: D, keyboard_parts:D_SOD123_axial, F.Cu at (376.6, -169.2)
- added D10: D, keyboard_parts:D_SOD123_axial, F.Cu at (356.6, -149.3)
- added D11: D, keyboard_parts:D_SOD123_axial, F.Cu at (376.6, -162.0)
- added D12: D, keyboard_parts:D_SOD123_axial, F.Cu at (356.6, -152.9)
- added D13: D, keyboard_parts:D_SOD123_axial, F.Cu at (376.6, -172.8)
- added D14: D, keyboard_parts:D_SOD123_axial, F.Cu at (336.7, -129.3)
- added D15: D, keyboard_parts:D_SOD123_axial, F.Cu at (347.1, -136.5)
- added D16: D, keyboard_parts:D_SOD123_axial, F.Cu at (336.7, -132.9)
- added D17: D, keyboard_parts:D_SOD123_axial, F.Cu at (376.6, -176.4)
- added D22: D, keyboard_parts:D_SOD123_axial, F.Cu at (356.6, -156.5)
- added D23: D, keyboard_parts:D_SOD123_axial, F.Cu at (336.7, -136.5)
- added D24: D, keyboard_parts:D_SOD123_axial, F.Cu at (367.0, -156.5)
- added D25: D, keyboard_parts:D_SOD123_axial, F.Cu at (256.9, -121.1)
- added K00: KEYSW, keebs:Mx_Alps_100, F.Cu at (16.5, -69.1)
- added K01: KEYSW, keebs:Mx_Alps_100, F.Cu at (35.6, -69.1)
- added K02: KEYSW, keebs:Mx_Alps_100, F.Cu at (54.6, -69.1)
- added K03: KEYSW, keebs:Mx_Alps_100, F.Cu at (73.7, -69.1)
- added K04: KEYSW, keebs:Mx_Alps_100, F.Cu at (130.8, -69.1)
- added K05: KEYSW, keebs:Mx_Alps_100, F.Cu at (149.9, -69.1)
- added K06: KEYSW, keebs:Mx_Alps_100, F.Cu at (168.9, -69.1)
- added K07: KEYSW, keebs:Mx_Alps_100, F.Cu at (188.0, -69.1)
- added K10: KEYSW, keebs:Mx_Alps_100, F.Cu at (361.4, -168.2)
- added K11: KEYSW, keebs:Mx_Alps_100, F.Cu at (321.5, -168.2)
- added K12: KEYSW, keebs:Mx_Alps_100, F.Cu at (281.7, -128.4)
- added K13: KEYSW, keebs:Mx_Alps_100, F.Cu at (340.4, -188.2)
- added K14: KEYSW, keebs:Mx_Alps_100, F.Cu at (301.6, -148.3)
- added K15: KEYSW, keebs:Mx_Alps_100, F.Cu at (320.5, -188.2)
- added K16: KEYSW, keebs:Mx_Alps_100, F.Cu at (281.7, -148.3)
- added K17: KEYSW, keebs:Mx_Alps_100, F.Cu at (301.6, -168.2)
- added K22: KEYSW, keebs:Mx_Alps_100, F.Cu at (281.7, -168.2)
- added K23: KEYSW, keebs:Mx_Alps_100, F.Cu at (300.6, -188.2)
- added K24: KEYSW, keebs:Mx_Alps_100, F.Cu at (261.7, -132.8)
- added K25: KEYSW, keebs:Mx_Alps_100, F.Cu at (280.6, -188.2)
- added REF**: MountingHole_3.2mm_M3_Pad, MountingHole:MountingHole_3.2mm_M3_Pad, F.Cu at (200.4, -86.6)
- added REF**: MountingHole_3.2mm_M3_Pad, MountingHole:MountingHole_3.2mm_M3_Pad, F.Cu at (154.9, -86.6)
- added REF**: MountingHole_3.2mm_M3_Pad, MountingHole:MountingHole_3.2mm_M3_Pad, F.Cu at (49.6, -86.6)
- added REF**: MountingHole_3.2mm_M3_Pad, MountingHole:MountingHole_3.2mm_M3_Pad, F.Cu at (4.07, -86.6)
- added REF**: MountingHole_3.2mm_M3_Pad, MountingHole:MountingHole_3.2mm_M3_Pad, F.Cu at (200.4, -4.07)
- added REF**: MountingHole_3.2mm_M3_Pad, MountingHole:MountingHole_3.2mm_M3_Pad, F.Cu at (154.8, -4.07)
- added REF**: MountingHole_3.2mm_M3_Pad, MountingHole:MountingHole_3.2mm_M3_Pad, F.Cu at (49.6, -4.07)
- added REF**: MountingHole_3.2mm_M3_Pad, MountingHole:MountingHole_3.2mm_M3_Pad, F.Cu at (4.07, -4.07)
Other:
- board outline added: 195 x 76.1 mm

Commit message: Add Size DWG for KiCad & Create PCB
Parts:
- removed K10: KEYSW, keebs:Mx_Alps_100
- moved D11 358.7 mm to (35.6, -50.8)
- moved D10 354.1 mm to (16.5, -50.8)
- moved D01 328.0 mm to (35.6, -79.4)
- moved D13 326.6 mm to (73.7, -50.8)
- moved D00 323.0 mm to (16.5, -79.4)
- moved D12 318.8 mm to (54.6, -50.8)
- moved D22 318.0 mm to (64.1, -31.8)
- moved K11 313.2 mm to (35.6, -40.5)
- moved K13 304.9 mm to (73.7, -40.5)
- moved D03 290.6 mm to (73.7, -79.4)
- moved D02 285.9 mm to (54.6, -79.4)
- moved D24 275.6 mm to (121.3, -31.8)
- moved D23 274.3 mm to (83.2, -31.8)
- moved K23 273.9 mm to (83.2, -21.5)
- moved K22 262.4 mm to (64.2, -21.6)
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Routing:
- net /row0: track 0.00 -> 230.0 mm
- net /row1: track 0.00 -> 219.2 mm, vias 0 -> 3
- net /col2: track 0.00 -> 141.4 mm, vias 0 -> 9
- net /col0: track 0.00 -> 137.5 mm, vias 0 -> 9
- net /col3: track 0.00 -> 127.3 mm, vias 0 -> 6
- net /col1: track 0.00 -> 125.7 mm, vias 0 -> 11
- net /col7: track 0.00 -> 124.5 mm, vias 0 -> 9
- net /col5: track 0.00 -> 116.4 mm, vias 0 -> 7
- net /col6: track 0.00 -> 106.3 mm, vias 0 -> 7
- net /col4: track 0.00 -> 99.7 mm, vias 0 -> 7
- net /row2: track 0.00 -> 89.7 mm, vias 0 -> 2
- net Net-(D07-Pad2): track 0.00 -> 6.28 mm
- net Net-(D25-Pad2): track 0.00 -> 6.03 mm
- net Net-(D24-Pad2): track 0.00 -> 6.03 mm
- net Net-(D23-Pad2): track 0.00 -> 6.03 mm
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Other:
- board size 195 x 76.1 mm -> 204.5 x 90.7 mm
